File: pcb/4x6_split_pcb.kicad_pcb (KiCad board)
At the start: 2 copper layers, 61 parts, among them SW0-0 MX, SW0-1 MX, SW0-2 MX, SW0-3 MX, SW1-0 MX, SW1-1 MX, SW1-2 MX, SW1-3 MX, SW2-0 MX, SW2-1 MX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

Commit message: details on the pull request descriptions.
Parts:
- removed U3: TRRS, keebio:TRRS-PJ-320A
- D0-0, D0-1, D0-2, D0-3, D1-0, D1-1, D1-2, D1-3, D2-0, D2-1, D2-2, D2-3, D3-0, D3-1, D3-2, D3-3, D4-0, D4-1, D4-2, D4-3, D5-0, D5-1, D5-2, D5-3: footprint keebio:Diode -> Keebio-Parts:Diode
- H0, H1, H2, H3, H4, H5, H6: footprint keebio:MountingHole -> Keebio-Parts:MountingHole
- R0, R1: footprint keebio:Resistor -> Keebio-Parts:Resistor
- SW0-0, SW0-1, SW0-2, SW0-3, SW1-0, SW1-1, SW1-2, SW1-3, SW2-0, SW2-1, SW2-2, SW2-3, SW3-0, SW3-1, SW3-2, SW3-3, SW4-0, SW4-1, SW4-2, SW4-3, SW5-0, SW5-1, SW5-2, SW5-3: footprint keebio:Triple-Dual-1u-LED -> Keebio-Parts:Triple-Dual-1u-LED
- SWRST-1: footprint keebio:SW_Tactile_SPST_Angled_MJTP1117 -> Keebio-Parts:SW_Tactile_SPST_Angled_MJTP1117
- U1: footprint keebio:ArduinoProMicro -> Keebio-Parts:ArduinoProMicro
- U2: footprint keebio:TRRS-PJ-320A -> Keebio-Parts:TRRS-PJ-320A
- moved R0 91.2 mm to (214.5, 84.8), turned to 270 degrees
- moved U2 58.7 mm to (234.7, 85.4), turned to 270 degrees
- moved R1 21.8 mm to (217.8, 84.8), turned to 270 degrees
Connections:
- SW0-0 pad 3: Net-(SW0-0-Pad3) -> (no net)
- SW0-0 pad 4: Net-(SW0-0-Pad4) -> (no net)
- SW0-1 pad 3: Net-(SW0-1-Pad3) -> (no net)
- SW0-1 pad 4: Net-(SW0-1-Pad4) -> (no net)
- SW0-2 pad 3: Net-(SW0-2-Pad3) -> (no net)
- SW0-2 pad 4: Net-(SW0-2-Pad4) -> (no net)
- SW0-3 pad 3: Net-(SW0-3-Pad3) -> (no net)
- SW0-3 pad 4: Net-(SW0-3-Pad4) -> (no net)
- SW1-0 pad 3: Net-(SW1-0-Pad3) -> (no net)
- SW1-0 pad 4: Net-(SW1-0-Pad4) -> (no net)
- SW1-1 pad 3: Net-(SW1-1-Pad3) -> (no net)
- SW1-1 pad 4: Net-(SW1-1-Pad4) -> (no net)
- SW1-2 pad 3: Net-(SW1-2-Pad3) -> (no net)
- SW1-2 pad 4: Net-(SW1-2-Pad4) -> (no net)
- SW1-3 pad 3: Net-(SW1-3-Pad3) -> (no net)
- SW1-3 pad 4: Net-(SW1-3-Pad4) -> (no net)
- SW2-0 pad 3: Net-(SW2-0-Pad3) -> (no net)
- SW2-0 pad 4: Net-(SW2-0-Pad4) -> (no net)
- SW2-1 pad 3: Net-(SW2-1-Pad3) -> (no net)
- SW2-1 pad 4: Net-(SW2-1-Pad4) -> (no net)
- SW2-2 pad 3: Net-(SW2-2-Pad3) -> (no net)
- SW2-2 pad 4: Net-(SW2-2-Pad4) -> (no net)
- SW2-3 pad 3: Net-(SW2-3-Pad3) -> (no net)
- SW2-3 pad 4: Net-(SW2-3-Pad4) -> (no net)
- SW3-0 pad 3: Net-(SW3-0-Pad3) -> (no net)
- SW3-0 pad 4: Net-(SW3-0-Pad4) -> (no net)
- SW3-1 pad 3: Net-(SW3-1-Pad3) -> (no net)
- SW3-1 pad 4: Net-(SW3-1-Pad4) -> (no net)
- SW3-2 pad 3: Net-(SW3-2-Pad3) -> (no net)
- SW3-2 pad 4: Net-(SW3-2-Pad4) -> (no net)
- SW3-3 pad 3: Net-(SW3-3-Pad3) -> (no net)
- SW3-3 pad 4: Net-(SW3-3-Pad4) -> (no net)
- SW4-0 pad 3: Net-(SW4-0-Pad3) -> (no net)
- SW4-0 pad 4: Net-(SW4-0-Pad4) -> (no net)
- SW4-1 pad 3: Net-(SW4-1-Pad3) -> (no net)
- SW4-1 pad 4: Net-(SW4-1-Pad4) -> (no net)
- SW4-2 pad 3: Net-(SW4-2-Pad3) -> (no net)
- SW4-2 pad 4: Net-(SW4-2-Pad4) -> (no net)
- SW4-3 pad 3: Net-(SW4-3-Pad3) -> (no net)
- SW4-3 pad 4: Net-(SW4-3-Pad4) -> (no net)
- SW5-0 pad 3: Net-(SW5-0-Pad3) -> (no net)
- SW5-0 pad 4: Net-(SW5-0-Pad4) -> (no net)
- SW5-1 pad 3: Net-(SW5-1-Pad3) -> (no net)
- SW5-1 pad 4: Net-(SW5-1-Pad4) -> (no net)
- SW5-2 pad 3: Net-(SW5-2-Pad3) -> (no net)
- SW5-2 pad 4: Net-(SW5-2-Pad4) -> (no net)
- SW5-3 pad 3: Net-(SW5-3-Pad3) -> (no net)
- SW5-3 pad 4: Net-(SW5-3-Pad4) -> (no net)
- U1 pad 1: Net-(U1-Pad1) -> (no net)
- U1 pad 13: Net-(U1-Pad13) -> (no net)
- U1 pad 14: Net-(U1-Pad14) -> (no net)
- U1 pad 2: Net-(U1-Pad2) -> (no net)
- U1 pad 23: +5V -> (no net)
- U1 pad 24: Net-(U1-Pad24) -> (no net)
- U1 pad 3: +5V -> (no net)
- U1 pad 4: +5V -> (no net)
- U1 pad 7: Net-(U1-Pad7) -> (no net)
- U1 pad 8: Net-(U1-Pad8) -> (no net)
Routing:
- net col0: track 0.00 -> 114.4 mm
- net Net-(D0-2-Pad2): track 0.00 -> 28.3 mm
- net Net-(D0-0-Pad2): track 0.00 -> 27.5 mm
- net Net-(D0-1-Pad2): track 0.00 -> 25.1 mm
- net Net-(D0-3-Pad2): track 0.00 -> 24.0 mm
