File: pcb/4x6_split_pcb.sch (KiCad schematic (older format))
At the start: 61 parts, among them SW0-0 MX, SW0-1 MX, SW0-2 MX, SW0-3 MX, SW1-0 MX, SW1-1 MX, SW1-2 MX, SW1-3 MX, SW2-0 MX, SW2-1 MX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

Commit message: details on the pull request descriptions.
Parts:
- removed U3: TRRS, keebio:TRRS-PJ-320A, symbol keebio_components:TRRS
- D0-0, D0-1, D0-2, D0-3, D1-0, D1-1, D1-2, D1-3, D2-0, D2-1, D2-2, D2-3, D3-0, D3-1, D3-2, D3-3, D4-0, D4-1, D4-2, D4-3, D5-0, D5-1, D5-2, D5-3: footprint keebio:Diode -> Keebio-Parts:Diode
- H0, H1, H2, H3, H4, H5, H6: footprint keebio:MountingHole -> Keebio-Parts:MountingHole; symbol keebio_components:Hole -> 4x6_split_pcb-rescue:Hole-keebio_components
- R0, R1: footprint keebio:Resistor -> Keebio-Parts:Resistor; symbol tmk_components:R -> 4x6_split_pcb-rescue:R-tmk_components
- SW0-0, SW0-1, SW0-2, SW0-3, SW1-0, SW1-1, SW1-2, SW1-3, SW2-0, SW2-1, SW2-2, SW2-3, SW3-0, SW3-1, SW3-2, SW3-3, SW4-0, SW4-1, SW4-2, SW4-3, SW5-0, SW5-1, SW5-2, SW5-3: footprint keebio:Triple-Dual-1u-LED -> Keebio-Parts:Triple-Dual-1u-LED; symbol keebio_components:MX -> 4x6_split_pcb-rescue:MX-keebio_components
- SWRST-1: footprint keebio:SW_Tactile_SPST_Angled_MJTP1117 -> Keebio-Parts:SW_Tactile_SPST_Angled_MJTP1117; symbol tmk_components:SW_PUSH -> 4x6_split_pcb-rescue:SW_PUSH-tmk_components
- U1: footprint keebio:ArduinoProMicro -> Keebio-Parts:ArduinoProMicro
- U2: footprint keebio:TRRS-PJ-320A -> Keebio-Parts:TRRS-PJ-320A; symbol keebio_components:TRRS -> 4x6_split_pcb-rescue:TRRS-keebio_components
Connections:
- net +5V: no longer U1.23 (GND), U1.3 (GND), U1.4 (GND)
